Commit message: implemented ros2_control for movement

File: wheelchair_description/urdf/chair.xacro (robot description, xacro)
@@ -2,5 +2,18 @@
 <robot name="wheelchair" xmlns:xacro="http://www.ros.org/wiki/xacro">
     <!-- base: to get robot position and details relative to the world-->
-    <link name="base_footprint"/>
+    <link name="world_root"/>
+    <link name="base_footprint">
+     <inertial>
+       <origin rpy="0.0 0.0 0.0" xyz="0.0 0.0 0.0"/>
+       <mass value="0.001"/>
+       <inertia ixx="0.00001" ixy="0.0" ixz="0.0" iyy="0.00001" iyz="0.0" izz="0.00001"/>
+     </inertial>
+    </link>
+    <!-- added this when i was getting kdl errors, why? -->
+    <joint name="world_root_to_footprint_joint" type="fixed">
+        <parent link="world_root"/>
+        <child link="base_footprint"/>
+        <origin rpy="0.0 0.0 0.0" xyz="0.0 0.0 0.0"/>
+    </joint>
     <!-- base_footprint to base_link -->
     <joint name="base_joint" type="fixed">
@@ -12,5 +25,5 @@
         <inertial>
             <origin xyz="0.0 0.0 0.0" rpy="0.0 0.0 0.0"/>
-            <mass value="0.0"/>
+            <mass value="15.0"/>
             <inertia ixx="0.1" ixy="0.0" ixz="0.0" iyy="0.1" iyz="0.0" izz="0.1"/>
         </inertial>
@@ -30,5 +43,5 @@
     <!-- The actual Wheelchair -->
     <!-- base to frame joint -->
-    <joint name="frame" type="fixed">
+    <joint name="frame_joint" type="fixed">
         <origin xyz="0.0 0.0 0.0" rpy="0.0 0.0 0.0"/>
         <parent link="base_link"/>
@@ -38,5 +51,5 @@
         <inertial>
             <origin xyz="0.0 0.0 0.0" rpy="0.0 0.0 0.0"/>
-            <mass value="0.0"/>
+            <mass value="1.0"/>
             <inertia ixx="0.01" ixy="0.0" ixz="0.0" iyy="0.01" iyz="0.0" izz="0.01"/>
         </inertial>
@@ -55,266 +68,272 @@
     </link>
     <!-- frame_to_seat -->
-    <joint name="seat" type="fixed">
+    <joint name="seat_joint" type="fixed">
         <origin xyz="0.0 -0.070 -0.038" rpy="0.0 0.0 0.0"/>
         <parent link="frame_link"/>
         <child link="seat_link"/>
         <!-- prismatic adds: Prevents math crashes by setting motion bounds (in meters) -->
+        <!-- <axis xyz="0 0 1"/>
+        <limit lower="-1.0" upper="1.0" effort="10.0" velocity="1.0"/> -->
+    </joint>
+    <link name="seat_link">
+        <inertial>
+            <origin xyz="0.0 0.0 0.0" rpy="0.0 0.0 0.0"/>
+            <mass value="1.0"/>
+            <inertia ixx="0.01" ixy="0.0" ixz="0.0" iyy="0.01" iyz="0.0" izz="0.01"/>
+        </inertial>
+        <visual>
+            <origin xyz="0.0 0.0 0.0" rpy="0.0 0.0 0.0"/>
+            <geometry>
+                <mesh filename="package://wheelchair_description/meshes/visual/seat_visual.obj"/>
+            </geometry>
+        </visual>
+        <collision>
+            <origin xyz="0.0 0.0 0.0" rpy="0.0 0.0 0.0"/>
+            <geometry>
+                <mesh filename="package://wheelchair_description/meshes/collision/seat_collision.stl"/>
+            </geometry>
+        </collision>
+    </link>
+    <!-- frame_to_back -->
+    <joint name="back_joint" type="fixed">
+        <origin xyz="0.0 -0.315 0.168" rpy="0.0 0.0 0.0"/>
+        <parent link="frame_link"/>
+        <child link="back_link"/>
+        <!-- prismatic adds: Prevents math crashes by setting motion bounds (in meters) -->
+        <!-- <axis xyz="0 0 1"/>
+        <limit lower="-1.0" upper="1.0" effort="10.0" velocity="1.0"/> -->
+    </joint>
+    <link name="back_link">
+        <inertial>
+            <origin xyz="0.0 0.0 0.0" rpy="0.0 0.0 0.0"/>
+            <mass value="1.0"/>
+            <inertia ixx="0.01" ixy="0.0" ixz="0.0" iyy="0.01" iyz="0.0" izz="0.01"/>
+        </inertial>
+        <visual>
+            <origin xyz="0.0 0.0 0.0" rpy="0.0 0.0 0.0"/>
+            <geometry>
+                <mesh filename="package://wheelchair_description/meshes/visual/back_visual.obj"/>
+            </geometry>
+        </visual>
+        <collision>
+            <origin xyz="0.0 0.0 0.0" rpy="0.0 0.0 0.0"/>
+            <geometry>
+                <mesh filename="package://wheelchair_description/meshes/collision/back_collision.stl"/>
+            </geometry>
+        </collision>
+    </link>
+    <!-- frame_to_left-panel -->
+    <joint name="left_panel_joint" type="fixed">
+        <origin xyz="-0.238 -0.100 0.044" rpy="0.0 0.0 0.0"/>
+        <parent link="frame_link"/>
+        <child link="left_panel_link"/>
+        <!-- prismatic adds: Prevents math crashes by setting motion bounds (in meters) -->
+        <!-- <axis xyz="0 1 0"/>
+        <limit lower="-1.0" upper="1.0" effort="10.0" velocity="1.0"/> -->
+    </joint>
+    <link name="left_panel_link">
+        <inertial>
+            <origin xyz="0.0 0.0 0.0" rpy="0.0 0.0 0.0"/>
+            <mass value="1.0"/>
+            <inertia ixx="0.01" ixy="0.0" ixz="0.0" iyy="0.01" iyz="0.0" izz="0.01"/>
+        </inertial>
+        <visual>
+            <origin xyz="0.0 0.0 0.0" rpy="0.0 0.0 0.0"/>
+            <geometry>
+                <mesh filename="package://wheelchair_description/meshes/visual/left_panel_visual.obj"/>
+            </geometry>
+        </visual>
+        <collision>
+            <origin xyz="0.0 0.0 0.0" rpy="0.0 0.0 0.0"/>
+            <geometry>
+                <mesh filename="package://wheelchair_description/meshes/collision/left_panel_collision.stl"/>
+            </geometry>
+        </collision>
+    </link>
+    <!-- frame_to_right-panel -->
+    <joint name="right_panel_joint" type="fixed">
+        <origin xyz="0.238 -0.100 0.043" rpy="0.0 0.0 0.0"/>
+        <parent link="frame_link"/>
+        <child link="right_panel_link"/>
+        <!-- prismatic adds: Prevents math crashes by setting motion bounds (in meters) -->
+        <!-- <axis xyz="0 0 1"/>
+        <limit lower="-1.0" upper="1.0" effort="10.0" velocity="1.0"/> -->
+    </joint>
+    <link name="right_panel_link">
+        <inertial>
+            <origin xyz="0.0 0.0 0.0" rpy="0.0 0.0 0.0"/>
+            <mass value="1.0"/>
+            <inertia ixx="0.01" ixy="0.0" ixz="0.0" iyy="0.01" iyz="0.0" izz="0.01"/>
+        </inertial>
+        <visual>
+            <origin xyz="0.0 0.0 0.0" rpy="0.0 0.0 0.0"/>
+            <geometry>
+                <mesh filename="package://wheelchair_description/meshes/visual/right_panel_visual.obj"/>
+            </geometry>
+        </visual>
+        <collision>
+            <origin xyz="0.0 0.0 0.0" rpy="0.0 0.0 0.0"/>
+            <geometry>
+                <mesh filename="package://wheelchair_description/meshes/collision/right_panel_collision.stl"/>
+            </geometry>
+        </collision>
+    </link>
+    <!-- frame_to_leftbackwheel -->
+    <joint name="leftbackwheel_joint" type="continuous">
+        <origin xyz="-0.276 -0.317 -0.194" rpy="0.0 0.0 0.0"/>
+        <parent link="frame_link"/>
+        <child link="leftbackwheel_link"/>
+        <!-- prismatic adds: Prevents math crashes by setting motion bounds (in meters) -->
+        <axis xyz="1 0 0"/>
+        <!-- <limit lower="-1.0" upper="1.0" effort="10.0" velocity="1.0"/> -->
+        <dynamics damping="0.1" friction="0.1"/>
+    </joint>
+    <link name="leftbackwheel_link">
+        <inertial>
+            <origin xyz="0.0 0.0 0.0" rpy="0.0 0.0 0.0"/>
+            <mass value="1.0"/>
+            <inertia ixx="0.01" ixy="0.0" ixz="0.0" iyy="0.01" iyz="0.0" izz="0.01"/>
+        </inertial>
+        <visual>
+            <origin xyz="0.0 0.0 0.0" rpy="0.0 0.0 0.0"/>
+            <geometry>
+                <mesh filename="package://wheelchair_description/meshes/visual/leftbackwheel_visual.obj"/>
+            </geometry>
+        </visual>
+        <collision>
+            <origin xyz="0.0 0.0 0.0" rpy="0.0 0.0 0.0"/>
+            <geometry>
+                <mesh filename="package://wheelchair_description/meshes/collision/leftbackwheel_collision.stl"/>
+            </geometry>
+        </collision>
+    </link>
+    <!-- frame_to_rightbackwheel -->
+    <joint name="rightbackwheel_joint" type="continuous">
+        <origin xyz="0.276 -0.317 -0.194" rpy="0.0 0.0 0.0"/>
+        <parent link="frame_link"/>
+        <child link="rightbackwheel_link"/>
+        <!-- prismatic adds: Prevents math crashes by setting motion bounds (in meters) -->
+        <axis xyz="1 0 0"/>
+        <!-- <limit lower="-1.0" upper="1.0" effort="10.0" velocity="1.0"/> -->
+        <dynamics damping="0.1" friction="0.1"/>
+    </joint>
+    <link name="rightbackwheel_link">
+        <inertial>
+            <origin xyz="0.0 0.0 0.0" rpy="0.0 0.0 0.0"/>
+            <mass value="1.0"/>
+            <inertia ixx="0.01" ixy="0.0" ixz="0.0" iyy="0.01" iyz="0.0" izz="0.01"/>
+        </inertial>
+        <visual>
+            <origin xyz="0.0 0.0 0.0" rpy="0.0 0.0 0.0"/>
+            <geometry>
+                <mesh filename="package://wheelchair_description/meshes/visual/rightbackwheel_visual.obj"/>
+            </geometry>
+        </visual>
+        <collision>
+            <origin xyz="0.0 0.0 0.0" rpy="0.0 0.0 0.0"/>
+            <geometry>
+                <mesh filename="package://wheelchair_description/meshes/collision/rightbackwheel_collision.stl"/>
+            </geometry>
+        </collision>
+    </link>
+    <!-- frame_to_left_caster -->
+    <joint name="left_caster_joint" type="continuous">
+        <origin xyz="-0.216 0.161 -0.314" rpy="0.0 0.0 0.0"/>
+        <parent link="frame_link"/>
+        <child link="left_caster_link"/>
+        <!-- prismatic adds: Prevents math crashes by setting motion bounds (in meters) -->
         <axis xyz="0 0 1"/>
-        <limit lower="-1.0" upper="1.0" effort="10.0" velocity="1.0"/>
-    </joint>
-    <link name="seat_link">
-        <inertial>
-            <origin xyz="0.0 0.0 0.0" rpy="0.0 0.0 0.0"/>
-            <mass value="0.0"/>
-            <inertia ixx="0.01" ixy="0.0" ixz="0.0" iyy="0.01" iyz="0.0" izz="0.01"/>
-        </inertial>
-        <visual>
-            <origin xyz="0.0 0.0 0.0" rpy="0.0 0.0 0.0"/>
-            <geometry>
-                <mesh filename="package://wheelchair_description/meshes/visual/seat_visual.obj"/>
-            </geometry>
-        </visual>
-        <collision>
-            <origin xyz="0.0 0.0 0.0" rpy="0.0 0.0 0.0"/>
-            <geometry>
-                <mesh filename="package://wheelchair_description/meshes/collision/seat_collision.stl"/>
-            </geometry>
-        </collision>
-    </link>
-    <!-- frame_to_back -->
-    <joint name="back" type="fixed">
-        <origin xyz="0.0 -0.315 0.168" rpy="0.0 0.0 0.0"/>
-        <parent link="frame_link"/>
-        <child link="back_link"/>
+        <!-- <limit lower="-1.0" upper="1.0" effort="10.0" velocity="1.0"/> -->
+        <dynamics damping="0.1" friction="0.1"/>
+    </joint>
+    <!-- casters only had stl format for whatever reason -->
+    <link name="left_caster_link">
+        <inertial>
+            <origin xyz="0.0 0.0 0.0" rpy="0.0 0.0 0.0"/>
+            <mass value="1.0"/>
+            <inertia ixx="0.01" ixy="0.0" ixz="0.0" iyy="0.01" iyz="0.0" izz="0.01"/>
+        </inertial>
+        <visual>
+            <origin xyz="0.0 0.0 0.0" rpy="0.0 0.0 0.0"/>
+            <geometry>
+                <mesh filename="package://wheelchair_description/meshes/visual/left_caster_visual.stl"/>
+            </geometry>
+        </visual>
+        <collision>
+            <origin xyz="0.0 0.0 0.0" rpy="0.0 0.0 0.0"/>
+            <geometry>
+                <mesh filename="package://wheelchair_description/meshes/collision/left_caster_collision.stl"/>
+            </geometry>
+        </collision>
+    </link>
+    <!-- frame_to_rightcaster -->
+    <joint name="right_caster_joint" type="continuous">
+        <origin xyz="0.216 0.161 -0.314" rpy="0.0 0.0 0.0"/>
+        <parent link="frame_link"/>
+        <child link="right_caster_link"/>
         <!-- prismatic adds: Prevents math crashes by setting motion bounds (in meters) -->
         <axis xyz="0 0 1"/>
-        <limit lower="-1.0" upper="1.0" effort="10.0" velocity="1.0"/>
-    </joint>
-    <link name="back_link">
-        <inertial>
-            <origin xyz="0.0 0.0 0.0" rpy="0.0 0.0 0.0"/>
-            <mass value="0.0"/>
-            <inertia ixx="0.01" ixy="0.0" ixz="0.0" iyy="0.01" iyz="0.0" izz="0.01"/>
-        </inertial>
-        <visual>
-            <origin xyz="0.0 0.0 0.0" rpy="0.0 0.0 0.0"/>
-            <geometry>
-                <mesh filename="package://wheelchair_description/meshes/visual/back_visual.obj"/>
-            </geometry>
-        </visual>
-        <collision>
-            <origin xyz="0.0 0.0 0.0" rpy="0.0 0.0 0.0"/>
-            <geometry>
-                <mesh filename="package://wheelchair_description/meshes/collision/back_collision.stl"/>
-            </geometry>
-        </collision>
-    </link>
-    <!-- frame_to_left-panel -->
-    <joint name="left_panel" type="fixed">
-        <origin xyz="-0.238 -0.100 0.044" rpy="0.0 0.0 0.0"/>
-        <parent link="frame_link"/>
-        <child link="left_panel"/>
-        <!-- prismatic adds: Prevents math crashes by setting motion bounds (in meters) -->
-        <axis xyz="0 1 0"/>
-        <limit lower="-1.0" upper="1.0" effort="10.0" velocity="1.0"/>
-    </joint>
-    <link name="left_panel">
-        <inertial>
-            <origin xyz="0.0 0.0 0.0" rpy="0.0 0.0 0.0"/>
-            <mass value="1.0"/>
-            <inertia ixx="0.01" ixy="0.0" ixz="0.0" iyy="0.01" iyz="0.0" izz="0.01"/>
-        </inertial>
-        <visual>
-            <origin xyz="0.0 0.0 0.0" rpy="0.0 0.0 0.0"/>
-            <geometry>
-                <mesh filename="package://wheelchair_description/meshes/visual/left_panel_visual.obj"/>
-            </geometry>
-        </visual>
-        <collision>
-            <origin xyz="0.0 0.0 0.0" rpy="0.0 0.0 0.0"/>
-            <geometry>
-                <mesh filename="package://wheelchair_description/meshes/collision/left_panel_collision.stl"/>
-            </geometry>
-        </collision>
-    </link>
-    <!-- frame_to_right-panel -->
-    <joint name="right_panel" type="fixed">
-        <origin xyz="0.238 -0.100 0.043" rpy="0.0 0.0 0.0"/>
-        <parent link="frame_link"/>
-        <child link="right_panel"/>
-        <!-- prismatic adds: Prevents math crashes by setting motion bounds (in meters) -->
-        <axis xyz="0 0 1"/>
-        <limit lower="-1.0" upper="1.0" effort="10.0" velocity="1.0"/>
-    </joint>
-    <link name="right_panel">
-        <inertial>
-            <origin xyz="0.0 0.0 0.0" rpy="0.0 0.0 0.0"/>
-            <mass value="1.0"/>
-            <inertia ixx="0.01" ixy="0.0" ixz="0.0" iyy="0.01" iyz="0.0" izz="0.01"/>
-        </inertial>
-        <visual>
-            <origin xyz="0.0 0.0 0.0" rpy="0.0 0.0 0.0"/>
-            <geometry>
-                <mesh filename="package://wheelchair_description/meshes/visual/right_panel_visual.obj"/>
-            </geometry>
-        </visual>
-        <collision>
-            <origin xyz="0.0 0.0 0.0" rpy="0.0 0.0 0.0"/>
-            <geometry>
-                <mesh filename="package://wheelchair_description/meshes/collision/right_panel_collision.stl"/>
-            </geometry>
-        </collision>
-    </link>
-    <!-- frame_to_leftbackwheel -->
-    <joint name="leftbackwheel" type="continuous">
-        <origin xyz="-0.276 -0.317 -0.194" rpy="0.0 0.0 0.0"/>
-        <parent link="frame_link"/>
-        <child link="leftbackwheel"/>
+        <!-- <limit lower="-1.0" upper="1.0" effort="10.0" velocity="1.0"/> -->
+        <dynamics damping="0.1" friction="0.1"/>
+    </joint>
+    <link name="right_caster_link">
+        <inertial>
+            <origin xyz="0.0 0.0 0.0" rpy="0.0 0.0 0.0"/>
+            <mass value="1.0"/>
+            <inertia ixx="0.01" ixy="0.0" ixz="0.0" iyy="0.01" iyz="0.0" izz="0.01"/>
+        </inertial>
+        <visual>
+            <origin xyz="0.0 0.0 0.0" rpy="0.0 0.0 0.0"/>
+            <geometry>
+                <mesh filename="package://wheelchair_description/meshes/visual/right_caster_visual.stl"/>
+            </geometry>
+        </visual>
+        <collision>
+            <origin xyz="0.0 0.0 0.0" rpy="0.0 0.0 0.0"/>
+            <geometry>
+                <mesh filename="package://wheelchair_description/meshes/collision/right_caster_collision.stl"/>
+            </geometry>
+        </collision>
+    </link>
+    <!-- left_caster_to_leftfrontwheel -->
+    <joint name="leftfrontwheel_joint" type="continuous">
+        <origin xyz="0.0 0.027 -0.086" rpy="0.0 0.0 0.0"/>
+        <parent link="left_caster_link"/>
+        <child link="leftfrontwheel_link"/>
         <!-- prismatic adds: Prevents math crashes by setting motion bounds (in meters) -->
         <axis xyz="1 0 0"/>
-        <limit lower="-1.0" upper="1.0" effort="10.0" velocity="1.0"/>
-    </joint>
-    <link name="leftbackwheel">
-        <inertial>
-            <origin xyz="0.0 0.0 0.0" rpy="0.0 0.0 0.0"/>
-            <mass value="1.0"/>
-            <inertia ixx="0.01" ixy="0.0" ixz="0.0" iyy="0.01" iyz="0.0" izz="0.01"/>
-        </inertial>
-        <visual>
-            <origin xyz="0.0 0.0 0.0" rpy="0.0 0.0 0.0"/>
-            <geometry>
-                <mesh filename="package://wheelchair_description/meshes/visual/leftbackwheel_visual.obj"/>
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