Commit message: obstacle detection_first iteration

File: wheelchair_description/urdf/chair.xacro (robot description, xacro)
@@ -1,5 +1,7 @@
 <?xml version="1.0"?>
 <robot name="wheelchair" xmlns:xacro="http://www.ros.org/wiki/xacro">
+    <xacro:include filename="chair_sensors.xacro" />
     <!-- base: to get robot position and details relative to the world-->
+    <!-- <link name="world"/> -->
     <link name="world_root"/>
     <link name="base_footprint">
@@ -20,5 +22,5 @@
         <parent link="base_footprint"/>
         <child link="base_link"/>
-        <origin xyz="0.0 0.0 0.0" rpy="0.0 0.0 0.0"/>
+        <origin xyz="0.0 -0.15 0.0" rpy="0.0 0.0 0.0"/>
     </joint>
     <link name="base_link">
@@ -185,5 +187,5 @@
         <child link="leftbackwheel_link"/>
         <!-- prismatic adds: Prevents math crashes by setting motion bounds (in meters) -->
-        <axis xyz="1 0 0"/>
+        <axis xyz="-1 0 0"/>
         <!-- <limit lower="-1.0" upper="1.0" effort="10.0" velocity="1.0"/> -->
         <dynamics damping="0.1" friction="0.1"/>
@@ -214,5 +216,5 @@
         <child link="rightbackwheel_link"/>
         <!-- prismatic adds: Prevents math crashes by setting motion bounds (in meters) -->
-        <axis xyz="1 0 0"/>
+        <axis xyz="-1 0 0"/>
         <!-- <limit lower="-1.0" upper="1.0" effort="10.0" velocity="1.0"/> -->
         <dynamics damping="0.1" friction="0.1"/>
@@ -578,4 +580,125 @@
         </collision>
     </link>
+<!-- obstacles -->
+    <!-- <joint name="world_to_world_root_joint" type="fixed">
+        <parent link="world"/>
+        <child link="world_root"/>
+        <origin rpy="0.0 0.0 0.0" xyz="0.0 0.0 0.0"/>
+    </joint>
+    <joint name="testing_pillar1_joint" type="fixed">
+        <origin xyz="2.0 0.0 1.5" rpy="0.0 0.0 0.0"/> <parent link="world"/>
+        <child link="testing_pillar1_link"/>
+    </joint>
+    <link name="testing_pillar1_link">
+        <inertial>
+            <mass value="50.0"/>
+            <inertia ixx="37.5" ixy="0.0" ixz="0.0" iyy="37.5" iyz="0.0" izz="0.1"/>
+        </inertial>
+        <visual>
+            <geometry>
+                <cylinder radius="0.15" length="3.0"/>
+            </geometry>
+            <material name="blue">
+                <color rgba="0.0 0.0 1.0 1.0"/>
+            </material>
+        </visual>
+        <collision>
+            <geometry>
+                <cylinder radius="0.15" length="3.0"/>
+            </geometry>
+        </collision>
+    </link>
+    <joint name="testing_pillar2_joint" type="fixed">
+        <origin xyz="6.0 0.0 1.5" rpy="0.0 0.0 0.0"/> <parent link="world"/>
+        <child link="testing_pillar2_link"/>
+    </joint>
+    <link name="testing_pillar2_link">
+        <inertial>
+            <mass value="50.0"/>
+            <inertia ixx="37.5" ixy="0.0" ixz="0.0" iyy="37.5" iyz="0.0" izz="0.1"/>
+        </inertial>
+        <visual>
+            <geometry>
+                <cylinder radius="0.15" length="3.0"/>
+            </geometry>
+            <material name="blue">
+                <color rgba="0.0 0.0 1.0 1.0"/>
+            </material>
+        </visual>
+        <collision>
+            <geometry>
+                <cylinder radius="0.15" length="3.0"/>
+            </geometry>
+        </collision>
+    </link>
+        <joint name="testing_pillar3_joint" type="fixed">
+        <origin xyz="10.0 0.0 1.5" rpy="0.0 0.0 0.0"/> <parent link="world"/>
+        <child link="testing_pillar3_link"/>
+    </joint>
+    <link name="testing_pillar3_link">
+        <inertial>
+            <mass value="50.0"/>
+            <inertia ixx="37.5" ixy="0.0" ixz="0.0" iyy="37.5" iyz="0.0" izz="0.1"/>
+        </inertial>
+        <visual>
+            <geometry>
+                <cylinder radius="0.15" length="3.0"/>
+            </geometry>
+            <material name="blue">
+                <color rgba="0.0 0.0 1.0 1.0"/>
+            </material>
+        </visual>
+        <collision>
+            <geometry>
+                <cylinder radius="0.15" length="3.0"/>
+            </geometry>
+        </collision>
+    </link>
+        <joint name="testing_pillar4_joint" type="fixed">
+        <origin xyz="4.0 4.0 1.5" rpy="0.0 0.0 0.0"/> <parent link="world"/>
+        <child link="testing_pillar4_link"/>
+    </joint>
+    <link name="testing_pillar4_link">
+        <inertial>
+            <mass value="50.0"/>
+            <inertia ixx="37.5" ixy="0.0" ixz="0.0" iyy="37.5" iyz="0.0" izz="0.1"/>
+        </inertial>
+        <visual>
+            <geometry>
+                <cylinder radius="0.15" length="3.0"/>
+            </geometry>
+            <material name="blue">
+                <color rgba="0.0 0.0 1.0 1.0"/>
+            </material>
+        </visual>
+        <collision>
+            <geometry>
+                <cylinder radius="0.15" length="3.0"/>
+            </geometry>
+        </collision>
+    </link>
+        <joint name="testing_pillar5_joint" type="fixed">
+        <origin xyz="12.0 1.0 1.5" rpy="0.0 0.0 0.0"/> <parent link="world"/>
+        <child link="testing_pillar5_link"/>
+    </joint>
+    <link name="testing_pillar5_link">
+        <inertial>
+            <mass value="50.0"/>
+            <inertia ixx="37.5" ixy="0.0" ixz="0.0" iyy="37.5" iyz="0.0" izz="0.1"/>
+        </inertial>
+        <visual>
+            <geometry>
+                <cylinder radius="0.15" length="3.0"/>
+            </geometry>
+            <material name="blue">
+                <color rgba="0.0 0.0 1.0 1.0"/>
+            </material>
+        </visual>
+        <collision>
+            <geometry>
+                <cylinder radius="0.15" length="3.0"/>
+            </geometry>
+        </collision>
+    </link> -->
 <!-- blue=up/down(z); green=front/back(y); red=left/right(x);  -->
     <!-- for ros2_control -->

File: wheelchair_description/urdf/chair_sensors.xacro (robot description, xacro)
@@ -1,5 +1,13 @@
 <?xml version="1.0" ?>
 <robot name="wheelchair" xmlns:xacro="http://www.ros.org/wiki/xacro">
-  <link name="lidar_pole_link">
+  <joint name="pole_joint" type="fixed">
+    <origin xyz="0.0 -0.362 0.205" rpy="0.0 0.0 0.0"/>
+    <parent link="frame_link"/>
+    <child link="pole_link"/>
+    <!-- prismatic add-ins -->
+    <!-- <axis xyz="0 0 0"/>
+    <limit lower="-1.0" upper="1.0" effort="10.0" velocity="1.0"/> -->
+  </joint>
+  <link name="pole_link">
     <inertial>
       <origin xyz="0.0 0.0 0.25" rpy="0.0 0.0 0.0"/>
@@ -22,13 +30,14 @@
     </collision>
   </link>
-  <joint name="lidar_pole_joint" type="fixed">
-    <origin xyz="0.0 -0.362 0.205" rpy="0.0 0.0 0.0"/>
-    <parent link="frame_link"/>
-    <child link="lidar_pole_link"/>
+<!-- pole to lidar -->
+  <joint name="lidar_joint" type="fixed">
+    <origin xyz="0.0 0.0 0.549" rpy="0.0 0.0 0.0"/>
+    <parent link="pole_link"/>
+    <child link="lidar_link"/>
     <!-- prismatic add-ins -->
-    <!-- <axis xyz="0 0 0"/>
-    <limit lower="-1.0" upper="1.0" effort="10.0" velocity="1.0"/> -->
+    <!-- <axis xyz="0 1 0" rpy="0 0 0"/> -->
+    <!-- <limit lower="-1.0" upper="1.0" effort="10.0" velocity="1.0"/> -->
   </joint>
-  <link name="laser_link">
+  <link name="lidar_link">
     <inertial>
       <origin xyz="0.0 0.0 0.0" rpy="0.0 0.0 0.0"/>
@@ -39,5 +48,5 @@
       <origin xyz="0.0 0.0 0.0" rpy="0.0 0.0 0.0"/>
       <geometry>
-        <box size="0.2 0.05 0.1"/>
+        <cylinder length="0.1" radius="0.06"/>
       </geometry>
       <material name="red">
@@ -48,20 +57,13 @@
       <origin xyz="0.0 0.0 0.0" rpy="0.0 0.0 0.0"/>
       <geometry>
-        <box size="0.05 0.2 0.1"/>
+        <cylinder length="0.1" radius="0.1"/>
       </geometry>
     </collision>
   </link>
-  <joint name="laser_joint" type="fixed">
-    <origin xyz="0.0 0.0 0.549" rpy="0.0 0.0 0.0"/>
-    <parent link="lidar_pole_link"/>
-    <child link="laser_link"/>
-    <!-- prismatic add-ins -->
-    <!-- <axis xyz="0  0"/>
-    <limit lower="-1.0" upper="1.0" effort="10.0" velocity="1.0"/>
-     -->
-  </joint>
-  <gazebo reference="laser_link">
+  <gazebo reference="lidar_link">
     <sensor type="gpu_lidar" name="generic_lidar">
-      <update_rate>10.0</update_rate> <topic>scan</topic>             <gz_frame_id>laser_link</gz_frame_id>
+      <update_rate>10.0</update_rate>
+      <topic>scan</topic>
+      <gz_frame_id>lidar_link</gz_frame_id>
       <lidar>
         <scan>
@@ -71,4 +73,9 @@
             <min_angle>-3.141592</min_angle> <max_angle>3.141592</max_angle>
           </horizontal>
+          <vertical>
+            <samples>64</samples>
+            <resolution>1</resolution>
+            <min_angle>-0.521799</min_angle> <max_angle>0.261799</max_angle>
+          </vertical>
         </scan>
         <range>

File: wheelchair_description/urdf/gazebo.xacro (robot description, xacro)
@@ -1,4 +1,5 @@
 <?xml version="1.0"?>
 <robot name="wheelchair" xmlns:xacro="http://www.ros.org/wiki/xacro">
+<!-- This whole file is to tell gazebo the things that move -->
     <!-- chair Wheels -->
     <!--
@@ -48,26 +49,26 @@
  movement and doesn't actually have its own -->
 <!-- chair Sensors -->
-<!-- 2D Laser Sensor -->
-<gazebo reference="laser_link">
+<!-- lidar Sensor -->
+<gazebo reference="lidar_link">
     <sensor name="lidar" type="gpu_lidar">
-        <pose>0 0 0 1.57 0 0</pose>
+        <pose relative_to='lidar_link'>0 0 0 0 0 0</pose>
         <always_on>true</always_on>
         <visualize>true</visualize>
         <topic>scan</topic>
-        <update_rate>5</update_rate>
-        <gz_frame_id>laser_link</gz_frame_id>
+        <update_rate>2</update_rate>
+        <gz_frame_id>lidar_link</gz_frame_id>
         <lidar>
             <scan>
                 <horizontal>
-                    <samples>10</samples>
+                    <samples>720</samples>
                     <resolution>1.00000</resolution>
-                    <min_angle>-1.00000</min_angle>
-                    <max_angle>0</max_angle>
+                    <min_angle>-3.14</min_angle>
+                    <max_angle>3.14</max_angle>
                 </horizontal>
             </scan>
             <range>
-                <min>0.05</min>
-                <max>4.0</max>
-                <resolution>0.02</resolution>
+                <min>0.01</min>
+                <max>12.0</max>
+                <resolution>0.005</resolution>
             </range>
             <noise>

Commit message: reduced lidar size

File: wheelchair_description/urdf/chair.xacro (robot description, xacro)
@@ -4,5 +4,18 @@
     <!-- base: to get robot position and details relative to the world-->
     <!-- <link name="world"/> -->
-    <link name="world_root"/>
+    <!-- added this when i was getting kdl errors, why? now i dont need it??-->
+    <!-- <joint name="world_to_footprint_joint" type="fixed">
+        <parent link="world"/>
+        <child link="base_footprint"/>
+        <origin rpy="0.0 0.0 0.0" xyz="0.0 0.0 0.0"/>
+    </joint> -->
+    <!-- <link name="world_root"/> -->
+    <!-- use this for rviz -->
+    <!-- <link name="odom"/>
+    <joint name="virtual_odom_joint" type="planar">
+        <parent link="odom"/>
+        <child link="base_footprint"/>
+        <origin xyz="0.0 0.0 0.0" rpy="0.0 0.0 0.0"/>
+    </joint> -->
     <link name="base_footprint">
      <inertial>
@@ -12,10 +25,4 @@
      </inertial>
     </link>
-    <!-- added this when i was getting kdl errors, why? -->
-    <joint name="world_root_to_footprint_joint" type="fixed">
-        <parent link="world_root"/>
-        <child link="base_footprint"/>
-        <origin rpy="0.0 0.0 0.0" xyz="0.0 0.0 0.0"/>
-    </joint>
     <!-- base_footprint to base_link -->
     <joint name="base_joint" type="fixed">

File: wheelchair_description/urdf/chair_sensors.xacro (robot description, xacro)
@@ -17,5 +17,5 @@
       <origin xyz="0.0 0.0 0.25" rpy="0.0 0.0 0.0"/>
       <geometry>
-        <cylinder radius="0.02" length="0.5"/>
+        <cylinder radius="0.016" length="0.5"/>
       </geometry>
       <material name="grey">
@@ -32,10 +32,10 @@
 <!-- pole to lidar -->
   <joint name="lidar_joint" type="fixed">
-    <origin xyz="0.0 0.0 0.549" rpy="0.0 0.0 0.0"/>
+    <origin xyz="0.0 0.0 0.522" rpy="0.0 0.0 0.0"/>
     <parent link="pole_link"/>
     <child link="lidar_link"/>
     <!-- prismatic add-ins -->
-    <!-- <axis xyz="0 1 0" rpy="0 0 0"/> -->
-    <!-- <limit lower="-1.0" upper="1.0" effort="10.0" velocity="1.0"/> -->
+    <!-- <axis xyz="0 0 1" rpy="0 0 0"/>
+    <limit lower="-1.0" upper="1.0" effort="10.0" velocity="1.0"/> -->
   </joint>
   <link name="lidar_link">
@@ -48,5 +48,5 @@
       <origin xyz="0.0 0.0 0.0" rpy="0.0 0.0 0.0"/>
       <geometry>
-        <cylinder length="0.1" radius="0.06"/>
+        <cylinder length="0.05" radius="0.05"/>
       </geometry>
       <material name="red">
